Commit message: Update plugin to support multiple realsense camera's

File: urdf/d435.gazebo.xacro (robot description, xacro)
@@ -6,7 +6,7 @@
 -->
 <robot xmlns:xacro="http://ros.org/wiki/xacro">
-  <xacro:macro name="simulation_d435" params="camera_name depth_optical_frame color_optical_frame infrared1_optical_frame infrared2_optical_frame" >
+  <xacro:macro name="simulation_d435" params="camera_name reference_link topics_ns depth_optical_frame color_optical_frame infrared1_optical_frame infrared2_optical_frame" >
     <!-- Load parameters to model's main link-->
-    <gazebo reference="camera_link">
+    <gazebo reference="${reference_link}">
       <self_collide>0</self_collide>
       <enable_wind>0</enable_wind>
@@ -22,5 +22,5 @@
       <!--<max_vel>0.01</max_vel>
       <min_depth>0</min_depth>-->
-      <sensor name="color" type="camera">
+      <sensor name="${camera_name}color" type="camera">
         <camera name="${camera_name}">
           <horizontal_fov>${69.4*deg_to_rad}</horizontal_fov>
@@ -44,5 +44,5 @@
         <visualize>1</visualize>
       </sensor>
-      <sensor name="ired1" type="camera">
+      <sensor name="${camera_name}ired1" type="camera">
         <camera name="${camera_name}">
           <horizontal_fov>${85.2*deg_to_rad}</horizontal_fov>
@@ -66,5 +66,5 @@
         <visualize>0</visualize>
       </sensor>
-      <sensor name="ired2" type="camera">
+      <sensor name="${camera_name}ired2" type="camera">
         <camera name="${camera_name}">
           <horizontal_fov>${85.2*deg_to_rad}</horizontal_fov>
@@ -88,5 +88,5 @@
         <visualize>0</visualize>
       </sensor>
-      <sensor name="depth" type="depth">
+      <sensor name="${camera_name}depth" type="depth">
         <camera name="${camera_name}">
           <horizontal_fov>${85.2*deg_to_rad}</horizontal_fov>
@@ -111,5 +111,6 @@
     </gazebo>
     <gazebo>
-      <plugin name="realsense_plugin" filename="librealsense_gazebo_plugin.so">
+      <plugin name="${topics_ns}" filename="librealsense_gazebo_plugin.so">
+        <prefix>${camera_name}</prefix>
       	<depthUpdateRate>60.0</depthUpdateRate>
       	<colorUpdateRate>60.0</colorUpdateRate>

File: urdf/d435.urdf.xacro (robot description, xacro)
@@ -6,7 +6,8 @@
 aluminum peripherial evaluation case.
 -->
-<robot xmlns:xacro="http://ros.org/wiki/xacro">
+<robot name="sensor_d435_gazebo" xmlns:xacro="http://ros.org/wiki/xacro">
+  <!--File includes-->
   <xacro:include filename="$(find realsense_gazebo_plugin)/urdf/d435.gazebo.xacro"/>
-  <xacro:macro name="sensor_d435" params="parent *origin">
+  <xacro:macro name="sensor_d435_gazebo" params="parent name:=camera topics_ns:=camera *origin">
     <xacro:property name="M_PI" value="3.1415926535897931" />
     <!-- The following values are approximate, and the camera node
@@ -27,23 +28,31 @@
     <xacro:property name="d435_cam_depth_py" value="0.0175"/>
     <xacro:property name="d435_cam_depth_pz" value="${d435_cam_height/2}"/>
-    <material name="aluminum">
+    <material name="${name}_aluminum">
 	  <color rgba="0.5 0.5 0.5 1"/>
     </material>
     <!-- camera body, with origin at bottom screw mount -->
-    <joint name="camera_joint" type="fixed">
+    <joint name="${name}_joint" type="fixed">
       <xacro:insert_block name="origin" />
       <parent link="${parent}"/>
-      <child link="camera_link" />
+      <child link="${name}_bottom_screw_frame" />
     </joint>
-    <link name="camera_link">
+    <link name="${name}_bottom_screw_frame"/>
+    <joint name="${name}_link_joint" type="fixed">
+      <origin xyz="0 ${d435_cam_depth_py} ${d435_cam_depth_pz}" rpy="0 0 0"/>
+      <parent link="${name}_bottom_screw_frame"/>
+      <child link="${name}_link" />
+    </joint>
+    <link name="${name}_link">
       <visual>
-      <origin xyz="${d435_cam_mount_from_center_offset} 0.0 ${d435_cam_height/2}" rpy="${M_PI/2} 0 ${M_PI/2}"/>
+      <origin xyz="${d435_cam_mount_from_center_offset} ${-d435_cam_depth_py} 0" rpy="${M_PI/2} 0 ${M_PI/2}"/>
         <geometry>
-	        <mesh filename="package://realsense_gazebo_plugin/meshes/d435.dae" />
+          <!-- <box size="${d435_cam_width} ${d435_cam_height} ${d435_cam_depth}"/> -->
+	  <mesh filename="package://realsense2_camera/meshes/d435.dae" />
+          <!--<mesh filename="package://realsense2_camera/meshes/d435/d435.dae" />-->
         </geometry>
-        <material name="aluminum"/>
+        <material name="${name}_aluminum"/>
       </visual>
       <collision>
-        <origin xyz="0.0 0.0 ${d435_cam_height/2}" rpy="0 0 0"/>
+        <origin xyz="0 ${-d435_cam_depth_py} 0" rpy="0 0 0"/>
         <geometry>
         <box size="${d435_cam_depth} ${d435_cam_width} ${d435_cam_height}"/>
@@ -58,72 +67,57 @@
     </link>
     <!-- camera depth joints and links -->
-    <joint name="camera_depth_joint" type="fixed">
-      <origin xyz="${d435_cam_depth_px} ${d435_cam_depth_py} ${d435_cam_depth_pz}" rpy="0 0 0"/>
-      <parent link="camera_link"/>
-      <child link="camera_depth_frame" />
+    <joint name="${name}_depth_joint" type="fixed">
+      <origin xyz="0 0 0" rpy="0 0 0"/>
+      <parent link="${name}_link"/>
+      <child link="${name}_depth_frame" />
     </joint>
-    <link name="camera_depth_frame"/>
-    <joint name="camera_depth_optical_joint" type="fixed">
+    <link name="${name}_depth_frame"/>
+    <joint name="${name}_depth_optical_joint" type="fixed">
       <origin xyz="0 0 0" rpy="${-M_PI/2} 0 ${-M_PI/2}" />
-      <parent link="camera_depth_frame" />
-      <child link="camera_depth_optical_frame" />
+      <parent link="${name}_depth_frame" />
+      <child link="${name}_depth_optical_frame" />
     </joint>
-    <link name="camera_depth_optical_frame"/>
+    <link name="${name}_depth_optical_frame"/>
     <!-- camera left IR joints and links -->
-    <joint name="camera_left_ir_joint" type="fixed">
+    <joint name="${name}_left_ir_joint" type="fixed">
       <origin xyz="0 ${d435_cam_depth_to_left_ir_offset} 0" rpy="0 0 0" />
-      <parent link="camera_depth_frame" />
-      <child link="camera_left_ir_frame" />
+      <parent link="${name}_depth_frame" />
+      <child link="${name}_left_ir_frame" />
     </joint>
-    <link name="camera_left_ir_frame"/>
-    <joint name="camera_left_ir_optical_joint" type="fixed">
+    <link name="${name}_left_ir_frame"/>
+    <joint name="${name}_left_ir_optical_joint" type="fixed">
       <origin xyz="0 0 0" rpy="${-M_PI/2} 0 ${-M_PI/2}" />
-      <parent link="camera_left_ir_frame" />
-      <child link="camera_left_ir_optical_frame" />
+      <parent link="${name}_left_ir_frame" />
+      <child link="${name}_left_ir_optical_frame" />
     </joint>
-    <link name="camera_left_ir_optical_frame"/>
+    <link name="${name}_left_ir_optical_frame"/>
     <!-- camera right IR joints and links -->
-    <joint name="camera_right_ir_joint" type="fixed">
+    <joint name="${name}_right_ir_joint" type="fixed">
       <origin xyz="0 ${d435_cam_depth_to_right_ir_offset} 0" rpy="0 0 0" />
-      <parent link="camera_depth_frame" />
-      <child link="camera_right_ir_frame" />
+      <parent link="${name}_depth_frame" />
+      <child link="${name}_right_ir_frame" />
     </joint>
-    <link name="camera_right_ir_frame"/>
-    <joint name="camera_right_ir_optical_joint" type="fixed">
+    <link name="${name}_right_ir_frame"/>
+    <joint name="${name}_right_ir_optical_joint" type="fixed">
       <origin xyz="0 0 0" rpy="${-M_PI/2} 0 ${-M_PI/2}" />
-      <parent link="camera_right_ir_frame" />
-      <child link="camera_right_ir_optical_frame" />
+      <parent link="${name}_right_ir_frame" />
+      <child link="${name}_right_ir_optical_frame" />
     </joint>
-    <link name="camera_right_ir_optical_frame"/>
+    <link name="${name}_right_ir_optical_frame"/>
     <!-- camera color joints and links -->
-    <joint name="camera_color_joint" type="fixed">
+    <joint name="${name}_color_joint" type="fixed">
       <origin xyz="0 ${d435_cam_depth_to_color_offset} 0" rpy="0 0 0" />
-      <parent link="camera_depth_frame" />
-      <child link="camera_color_frame" />
+      <parent link="${name}_depth_frame" />
+      <child link="${name}_color_frame" />
     </joint>
-    <link name="camera_color_frame">
-      <inertial>
-        <mass value="0.01" />
-        <origin xyz="0 0 0" rpy="0 0 0"/>
-        <inertia ixx="0.0"  ixy="0.0"  ixz="0.0"
-                 iyy="0.0"  iyz="0.0"
-                 izz="0.0" />
-      </inertial>
-    </link>
-    <joint name="camera_color_optical_joint" type="fixed">
+    <link name="${name}_color_frame"/>
+    <joint name="${name}_color_optical_joint" type="fixed">
       <origin xyz="0 0 0" rpy="${-M_PI/2} 0 ${-M_PI/2}" />
-      <parent link="camera_color_frame" />
-      <child link="camera_color_optical_frame" />
+      <parent link="${name}_color_frame" />
+      <child link="${name}_color_optical_frame" />
     </joint>
-    <link name="camera_color_optical_frame">
-      <inertial>
-        <mass value="0.01" />
-        <origin xyz="0 0 0" rpy="0 0 0"/>
-        <inertia ixx="0.0"  ixy="0.0"  ixz="0.0"
-                 iyy="0.0"  iyz="0.0"
-                 izz="0.0" />
-      </inertial>
-    </link>
-    <xacro:simulation_d435 camera_name="realsense" depth_optical_frame="camera_depth_optical_frame" color_optical_frame="camera_color_optical_frame" infrared1_optical_frame="camera_left_ir_optical_frame" infrared2_optical_frame="camera_right_ir_optical_frame"/>
+    <link name="${name}_color_optical_frame"/>
+    <!-- Realsense Gazebo Plugin -->
+    <xacro:simulation_d435 camera_name="${name}" reference_link="${name}_link" topics_ns="${topics_ns}" depth_optical_frame="${name}_depth_optical_frame" color_optical_frame="${name}_color_optical_frame" infrared1_optical_frame="${name}_left_ir_optical_frame" infrared2_optical_frame="${name}_right_ir_optical_frame"/>
   </xacro:macro>
 </robot>
