Commit message: Rm unnecessary files

File: urdf/d435.urdf.xacro (robot description, xacro)
@@ -40,5 +40,5 @@
       <origin xyz="${d435_cam_mount_from_center_offset} 0.0 ${d435_cam_height/2}" rpy="${M_PI/2} 0 ${M_PI/2}"/>
         <geometry>
-	        <mesh filename="package://realsense_gazebo_plugin/models/realsense_camera/meshes/d435.dae" />
+	        <mesh filename="package://realsense_gazebo_plugin/meshes/d435.dae" />
         </geometry>
         <material name="aluminum"/>

Commit message: fixed the issue with mesh location

File: urdf/d435.urdf.xacro (robot description, xacro)
@@ -48,6 +48,6 @@
         <geometry>
           <!-- <box size="${d435_cam_width} ${d435_cam_height} ${d435_cam_depth}"/> -->
-	  <mesh filename="package://realsense2_camera/meshes/d435.dae" />
-          <!--<mesh filename="package://realsense2_camera/meshes/d435/d435.dae" />-->
+          <mesh filename="package://realsense_gazebo_plugin/meshes/d435.dae" />
+          <!--<mesh filename="package://realsense_gazebo_plugin/meshes/d435/d435.dae" />-->
         </geometry>
         <material name="${name}_aluminum"/>
