Commit message: Added the topic_ns param for the t265 camera

File: urdf/t265.urdf.xacro (robot description, xacro)
@@ -8,5 +8,5 @@
 <robot name="sensor_t265_gazebo" xmlns:xacro="http://ros.org/wiki/xacro">
   <!--File includes-->
-  <xacro:macro name="sensor_t265_gazebo" params="parent name:=camera *origin">
+  <xacro:macro name="sensor_t265_gazebo" params="parent name:=camera topics_ns:=camera *origin">
     <xacro:property name="M_PI" value="3.1415926535897931" />
     <!-- The following values are approximate, and the camera node

Commit message: Add gazebo for t265

File: urdf/t265.urdf.xacro (robot description, xacro)
@@ -8,4 +8,5 @@
 <robot name="sensor_t265_gazebo" xmlns:xacro="http://ros.org/wiki/xacro">
   <!--File includes-->
+  <xacro:include filename="$(find realsense_gazebo_plugin)/urdf/t265.gazebo.xacro"/>
   <xacro:macro name="sensor_t265_gazebo" params="parent name:=camera topics_ns:=camera *origin">
     <xacro:property name="M_PI" value="3.1415926535897931" />
@@ -21,11 +22,11 @@
       <color rgba="0.5 0.5 0.5 1"/>
     </material>
-    <!-- camera body, with origin at camera_pose_frame -->
+    <!-- camera body, with origin at camera_link -->
     <joint name="${name}_pose_joint" type="fixed">
       <xacro:insert_block name="origin" />
       <parent link="${parent}"/>
-      <child link="${name}_pose_frame" />
+      <child link="${name}_link" />
     </joint>
-    <link name="${name}_pose_frame">
+    <link name="${name}_link">
       <visual>
       <origin xyz="0 0 0" rpy="0 0 0"/>
@@ -48,20 +49,32 @@
       </inertial>
     </link>
-    <joint name="${name}_fisheye2_joint" type="fixed">
-      <origin xyz="${fisheye2_offset_x} ${fisheye2_offset_y} ${fisheye2_offset_z}" rpy="${M_PI} 0 0"/>
-      <parent link="${name}_pose_frame"/>
+    <joint name="${name}_fisheye1_rgb_joint" type="fixed">
+      <origin xyz="${fisheye1_offset_x} ${fisheye1_offset_y} ${fisheye1_offset_z}" rpy="0 ${M_PI/2} ${M_PI/2}"/>
+      <parent link="${name}_link"/>
+      <child link="${name}_fisheye1_rgb_frame" />
+    </joint>
+    <link name="${name}_fisheye1_rgb_frame"/>
+    <joint name="${name}_fisheye2_rgb_joint" type="fixed">
+      <origin xyz="${fisheye2_offset_x} ${fisheye2_offset_y} ${fisheye2_offset_z}" rpy="0 ${M_PI/2} ${M_PI/2}"/>
+      <parent link="${name}_link"/>
+      <child link="${name}_fisheye2_rgb_frame" />
+    </joint>
+    <link name="${name}_fisheye2_rgb_frame"/>
+    <joint name="${name}_fisheye1_optical_joint" type="fixed">
+      <origin xyz="0 0 0" rpy="${M_PI/2} -${M_PI/2} ${M_PI/2}"/>
+      <parent link="${name}_fisheye1_rgb_frame"/>
+      <child link="${name}_fisheye1_optical_frame" />
+    </joint>
+    <link name="${name}_fisheye1_optical_frame"/>
+    <joint name="${name}_fisheye2_optical_joint" type="fixed">
+      <origin xyz="0 0 0" rpy="${M_PI/2} -${M_PI/2} ${M_PI/2}"/>
+      <parent link="${name}_fisheye2_rgb_frame"/>
       <child link="${name}_fisheye2_optical_frame" />
     </joint>
     <link name="${name}_fisheye2_optical_frame"/>
-    <joint name="${name}_fisheye1_joint" type="fixed">
-      <origin xyz="${fisheye1_offset_x} ${fisheye1_offset_y} ${fisheye1_offset_z}" rpy="${M_PI} 0 0"/>
-      <parent link="${name}_pose_frame"/>
-      <child link="${name}_fisheye1_optical_frame" />
-    </joint>
-    <link name="${name}_fisheye1_optical_frame"/>
     <!-- camera depth joints and links -->
     <joint name="${name}_gyro_optical_joint" type="fixed">
       <origin xyz="-0.0311 0 0.00655" rpy="0 ${M_PI} 0"/>
-      <parent link="${name}_pose_frame"/>
+      <parent link="${name}_link"/>
       <child link="${name}_gyro_optical_frame" />
     </joint>
@@ -73,4 +86,6 @@
     </joint>
     <link name="${name}_accel_optical_frame"/>
+    <!-- Realsense Gazebo Plugin -->
+    <xacro:simulation_t265 camera_name="${name}" fisheye1_reference_link="${name}_fisheye1_rgb_frame" fisheye2_reference_link="${name}_fisheye2_rgb_frame" topics_ns="${topics_ns}" fisheye1_optical_frame="${name}_fisheye1_optical_frame" fisheye2_optical_frame="${name}_fisheye2_optical_frame"/>
   </xacro:macro>
 </robot>
