Commit message: First version of working fisheye

File: urdf/t265.gazebo.xacro (robot description, xacro)
@@ -22,5 +22,5 @@
       <!--<max_vel>0.01</max_vel>
       <min_depth>0</min_depth>-->
-      <sensor name="${camera_name}fisheye1" type="camera">
+      <sensor name="${camera_name}fisheye1" type="wideanglecamera">
         <origin xyz="0 0 0" rpy="0 ${M_PI/2} 0" />
         <update_rate>30</update_rate>
@@ -35,14 +35,32 @@
             <far>100</far>
           </clip>
-          <distortion>
-            <k1>-0.00040996368625201285</k1>
-            <k2>0.03653175011277199</k2>
-            <k3>0.0</k3>
-            <p1>-0.034823670983314514</p1>
-            <p2>0.0052825710736215115</p2>
-            <center>0.5 0.5</center>
-          </distortion>
+         <lens>
+            <!-- type element is mandatory -->
+            <type>custom</type>
+            <!-- manually defined mapping function r = c1*f*fun(theta/c2 + c3) -->
+            <!-- More information here: https://en.wikipedia.org/wiki/Fisheye_lens#Mapping_function -->
+            <custom_function>
+              <c1>1.05</c1>   <!-- linear scaling -->
+              <c2>4</c2>      <!-- angle scaling -->
+              <f>1.0</f>      <!-- one more scaling parameter -->
+              <fun>tan</fun>  <!-- one of sin,tan,id -->
+            </custom_function>
+            <!-- if it is set to `true` your horizontal FOV will remain as defined -->
+            <!-- othervise it depends on lens type and custom function, if there is one -->
+            <scale_to_hfov>true</scale_to_hfov>
+            <!-- clip everything that is outside of this angle -->
+            <cutoff_angle>3.1415</cutoff_angle>
+            <!-- resolution of the cubemap texture, the highter it is - the sharper is your image -->
+            <env_texture_size>512</env_texture_size>
+          </lens>
+          <!--<distortion>-->
+            <!--<k1>-0.00040996368625201285</k1>-->
+            <!--<k2>0.03653175011277199</k2>-->
+            <!--<k3>0.0</k3>-->
+            <!--<p1>-0.034823670983314514</p1>-->
+            <!--<p2>0.0052825710736215115</p2>-->
+            <!--<center>0.5 0.5</center>-->
+          <!--</distortion>-->
         </camera>
-        <always_on>1</always_on>
         <plugin name="${camera_name}fisheye1" filename="libgazebo_ros_camera.so">
           <alwaysOn>true</alwaysOn>
@@ -58,9 +76,4 @@
           <distortionP1>-0.034823670983314514</distortionP1>
           <distortionP2>0.0052825710736215115</distortionP2>
-          <!--<distortionK1>0.0</distortionK1>-->
-          <!--<distortionK2>0.0</distortionK2>-->
-          <!--<distortionK3>0.0</distortionK3>-->
-          <!--<distortionT1>0.0</distortionT1>-->
-          <!--<distortionT2>0.0</distortionT2>-->
         </plugin>
       </sensor>
@@ -80,5 +93,5 @@
       <!--<max_vel>0.01</max_vel>
       <min_depth>0</min_depth>-->
-      <sensor name="${camera_name}fisheye2" type="camera">
+      <sensor name="${camera_name}fisheye2" type="wideanglecamera">
         <origin xyz="0 0 0" rpy="0 ${M_PI/2} 0" />
         <update_rate>30</update_rate>
@@ -93,12 +106,31 @@
             <far>100</far>
           </clip>
-          <distortion>
-            <k1>-0.00040996368625201285</k1>
-            <k2>0.03653175011277199</k2>
-            <k3>0.0</k3>
-            <p1>-0.034823670983314514</p1>
-            <p2>0.0052825710736215115</p2>
-            <center>0.5 0.5</center>
-          </distortion>
+         <lens>
+            <!-- type element is mandatory -->
+            <type>custom</type>
+            <!-- manually defined mapping function r = c1*f*fun(theta/c2 + c3) -->
+            <!-- More information here: https://en.wikipedia.org/wiki/Fisheye_lens#Mapping_function -->
+            <custom_function>
+              <c1>1.05</c1>   <!-- linear scaling -->
+              <c2>4</c2>      <!-- angle scaling -->
+              <f>1.0</f>      <!-- one more scaling parameter -->
+              <fun>tan</fun>  <!-- one of sin,tan,id -->
+            </custom_function>
+            <!-- if it is set to `true` your horizontal FOV will remain as defined -->
+            <!-- othervise it depends on lens type and custom function, if there is one -->
+            <scale_to_hfov>true</scale_to_hfov>
+            <!-- clip everything that is outside of this angle -->
+            <cutoff_angle>3.1415</cutoff_angle>
+            <!-- resolution of the cubemap texture, the highter it is - the sharper is your image -->
+            <env_texture_size>512</env_texture_size>
+          </lens>
+          <!--<distortion>-->
+            <!--<k1>-0.00040996368625201285</k1>-->
+            <!--<k2>0.03653175011277199</k2>-->
+            <!--<k3>0.0</k3>-->
+            <!--<p1>-0.034823670983314514</p1>-->
+            <!--<p2>0.0052825710736215115</p2>-->
+            <!--<center>0.5 0.5</center>-->
+          <!--</distortion>-->
         </camera>
         <always_on>1</always_on>
@@ -116,9 +148,4 @@
           <distortionP1>-0.034823670983314514</distortionP1>
           <distortionP2>0.0052825710736215115</distortionP2>
-          <!--<distortionK1>0.0</distortionK1>-->
-          <!--<distortionK2>0.0</distortionK2>-->
-          <!--<distortionK3>0.0</distortionK3>-->
-          <!--<distortionT1>0.0</distortionT1>-->
-          <!--<distortionT2>0.0</distortionT2>-->
         </plugin>
       </sensor>

File: urdf/t265.urdf.xacro (robot description, xacro)
@@ -62,5 +62,5 @@
     <link name="${name}_fisheye2_rgb_frame"/>
     <joint name="${name}_fisheye1_optical_joint" type="fixed">
-      <origin xyz="0 0 0" rpy="${M_PI/2} -${M_PI/2} ${M_PI/2}"/>
+      <origin xyz="0 0 0" rpy="-${M_PI/2} 0 -${M_PI/2}"/>
       <parent link="${name}_fisheye1_rgb_frame"/>
       <child link="${name}_fisheye1_optical_frame" />
@@ -68,5 +68,5 @@
     <link name="${name}_fisheye1_optical_frame"/>
     <joint name="${name}_fisheye2_optical_joint" type="fixed">
-      <origin xyz="0 0 0" rpy="${M_PI/2} -${M_PI/2} ${M_PI/2}"/>
+      <origin xyz="0 0 0" rpy="-${M_PI/2} 0 -${M_PI/2}"/>
       <parent link="${name}_fisheye2_rgb_frame"/>
       <child link="${name}_fisheye2_optical_frame" />
